File: keyswitches.kicad_sch (KiCad schematic)
At the start: 79 parts, among them U10 KEY_LARR, U11 KEY_STOP, U12 KEY_SPACE, U13 KEY_Q, U14 KEY_1, U15 KEY_SHIFTLOCK, U16 KEY_LSHIFT, U17 KEY_ESC, U18 KEY_>, U19 KEY_A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

Commit message: tweak PCB appearance
Parts:
- renumbered R13 to R?, R14 to R?, U19 to U?, U68 to U?, U67 to U?, U78 to U?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

Commit message: improve keyswitch footprint to show key IDs
Parts:
- gave numbers to parts that had none: 79
